File: PCB/peeko.kicad_pcb (KiCad board)
At the start: 2 copper layers, 21.8 x 51.3 mm, 6 parts, among them J1 Rasberry PI Pico, J2 Conn_02x15_Odd_Even, J3 Conn_01x02_Pin, J4 Conn_01x02_Pin

Commit message: level shifter
Other:
- board text added: "2 1"
- board text added: "30 29"
Changed lines of the file:
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@@
 		(tags "Through hole angled pin header THT 1x02 2.54mm single row")
 		(property "Reference" "J3"
-			(at 5.207 -1.143 270)
+			(at 5.207 -1.143 -90)
 			(unlocked yes)
 			(layer "B.SilkS")
@@
 		(tags "Through hole angled pin header THT 1x02 2.54mm single row")
 		(property "Reference" "J4"
-			(at 5.207 -1.397 270)
+			(at 5.207 -1.397 -90)
 			(unlocked yes)
 			(layer "B.SilkS")
@@
 		)
 	)
+	(gr_text "30\n\n29"
+		(at 158.75 85.217 270)
+		(layer "B.SilkS")
+		(effects
+			(font
+				(size 0.8 1)
+				(thickness 0.15)
+			)
+			(justify left mirror)
+		)
+	)
 	(gr_text "CHAIN"
 		(at 152.4 115.697 -90)
@@
 		)
 	)
+	(gr_text "2\n\n1"
+		(at 158.75 123.063 270)
+		(layer "B.SilkS")
+		(effects
+			(font
+				(size 0.8 1)
+				(thickness 0.15)
+			)
+			(justify right mirror)
+		)
+	)
