File: PCB/peeko_jy.kicad_pcb (KiCad board)
At the start: 4 copper layers, 52.1 x 45.7 mm, 60 parts, among them J1 Raspberry Pi Pico, J2 2x15x2.54mm_edge, J3 1x2x2.54mm, J4 1x2x2.54mm

Commit message: annotation
Parts:
- renumbered D25 to D1, D1 to D2

Commit message: schematic for JY board, remove all but PCBs
Parts:
- D1, D12, D2: footprint AnalyzerBoxPCB_fork:SC-59 -> 000_LOCAL:SC-59
- D10, D11, D13, D14, D15, D16, D17, D18, D19, D20, D21, D22, D23, D24, D3, D4, D5, D6, D7, D8, D9: value (none) -> BAV99; footprint AnalyzerBoxPCB_fork:SC-59 -> 000_LOCAL:SC-59
- D25: renamed from D31; footprint AnalyzerBoxPCB_fork:SC-59 -> 000_LOCAL:SC-59
- J1: value Raspberry Pi Pico -> Rasberry PI Pico; footprint AnalyzerBoxPCB_fork:Raspberry Pi Pico -> 000_LOCAL:dip-40-700-pi-pico
- J2: value 2x15x2.54mm_edge -> Conn_02x15_Odd_Even; footprint AnalyzerBoxPCB_fork:HDR-TH_30P-P2.54-V-F-R2-C15-S2.54-A -> 000_LOCAL:IDC_02x15_2.54_THT_male_pcb_edge
- J3, J4: value 1x2x2.54mm -> Conn_01x02_Pin
- R1: renamed from R2; footprint AnalyzerBoxPCB_fork:R_0805 -> 000_LOCAL:R_0805
- R10: renamed from R11; value (none) -> 220; footprint AnalyzerBoxPCB_fork:R_0805 -> 000_LOCAL:R_0805
- R11: renamed from R12; value (none) -> 220; footprint AnalyzerBoxPCB_fork:R_0805 -> 000_LOCAL:R_0805
- R12: renamed from R13; footprint AnalyzerBoxPCB_fork:R_0805 -> 000_LOCAL:R_0805
- R13: renamed from R25; value (none) -> 220; footprint AnalyzerBoxPCB_fork:R_0805 -> 000_LOCAL:R_0805
- R14: renamed from R24; value (none) -> 220; footprint AnalyzerBoxPCB_fork:R_0805 -> 000_LOCAL:R_0805
- R15: renamed from R23; value (none) -> 220; footprint AnalyzerBoxPCB_fork:R_0805 -> 000_LOCAL:R_0805
- R16: renamed from R22; value (none) -> 220; footprint AnalyzerBoxPCB_fork:R_0805 -> 000_LOCAL:R_0805
- R17: renamed from R21; value (none) -> 220; footprint AnalyzerBoxPCB_fork:R_0805 -> 000_LOCAL:R_0805
- R18: renamed from R20; value (none) -> 220; footprint AnalyzerBoxPCB_fork:R_0805 -> 000_LOCAL:R_0805
- R19: value (none) -> 220; footprint AnalyzerBoxPCB_fork:R_0805 -> 000_LOCAL:R_0805
- R2: renamed from R3; value (none) -> 220; footprint AnalyzerBoxPCB_fork:R_0805 -> 000_LOCAL:R_0805
- R20: renamed from R18; value (none) -> 220; footprint AnalyzerBoxPCB_fork:R_0805 -> 000_LOCAL:R_0805
- R21: renamed from R17; value (none) -> 220; footprint AnalyzerBoxPCB_fork:R_0805 -> 000_LOCAL:R_0805
- R22: renamed from R16; value (none) -> 220; footprint AnalyzerBoxPCB_fork:R_0805 -> 000_LOCAL:R_0805
- R23: renamed from R15; value (none) -> 220; footprint AnalyzerBoxPCB_fork:R_0805 -> 000_LOCAL:R_0805
- R24: renamed from R14; value (none) -> 220; footprint AnalyzerBoxPCB_fork:R_0805 -> 000_LOCAL:R_0805
- R25: renamed from R1; value 100K -> 100k; footprint AnalyzerBoxPCB_fork:R_0805 -> 000_LOCAL:R_0805
- R3: renamed from R4; value (none) -> 220; footprint AnalyzerBoxPCB_fork:R_0805 -> 000_LOCAL:R_0805
- R4: renamed from R5; value (none) -> 220; footprint AnalyzerBoxPCB_fork:R_0805 -> 000_LOCAL:R_0805
- R5: renamed from R6; value (none) -> 220; footprint AnalyzerBoxPCB_fork:R_0805 -> 000_LOCAL:R_0805
- R6: renamed from R7; value (none) -> 220; footprint AnalyzerBoxPCB_fork:R_0805 -> 000_LOCAL:R_0805
- R7: renamed from R8; value (none) -> 220; footprint AnalyzerBoxPCB_fork:R_0805 -> 000_LOCAL:R_0805
- R8: renamed from R9; value (none) -> 220; footprint AnalyzerBoxPCB_fork:R_0805 -> 000_LOCAL:R_0805
- R9: renamed from R10; value (none) -> 220; footprint AnalyzerBoxPCB_fork:R_0805 -> 000_LOCAL:R_0805
- turned R13 to -90 degrees
- turned R14 to -90 degrees
- turned R15 to -90 degrees
- turned R16 to -90 degrees
- turned R17 to -90 degrees
- turned R18 to -90 degrees
- turned R19 to -90 degrees
- turned R20 to -90 degrees
- turned R21 to -90 degrees
- turned R22 to -90 degrees
- turned R23 to -90 degrees
- turned R24 to -90 degrees
Connections:
- net $1N6412 renamed /CH0
- net $1N6457 renamed /CH1
- net $1N6576 renamed /CH2
- net $1N6580 renamed /CH3
- net $1N6666 renamed /CH4
- net $1N6670 renamed /CH5
- net $1N6756 renamed /CH6
- net $1N6760 renamed /CH7
- net $1N6846 renamed /CH8
- net $1N6850 renamed /CH9
- net $1N6936 renamed /CH10
- net $1N6940 renamed /CH11
- net +3.3V renamed +3V3
- net CHAN_0 renamed /_CH0
- net CHAN_1 renamed /_CH1
- net CHAN_10 renamed /_CH10
- net CHAN_11 renamed /_CH11
- net CHAN_2 renamed /_CH2
- net CHAN_3 renamed /_CH3
- net CHAN_4 renamed /_CH4
- net CHAN_5 renamed /_CH5
- net CHAN_6 renamed /_CH6
- net CHAN_7 renamed /_CH7
- net CHAN_8 renamed /_CH8
- net CHAN_9 renamed /_CH9
- net EXT_CHAIN renamed /CHAIN
- net EXT_T renamed /TRIGGER
- D13 pad 3: CHAN_12 -> /_CH12
- D14 pad 3: CHAN_13 -> /_CH13
- D15 pad 3: CHAN_14 -> /_CH14
- D16 pad 3: CHAN_15 -> /_CH15
- D17 pad 3: CHAN_16 -> /_CH16
- D18 pad 3: CHAN_17 -> /_CH17
- D19 pad 3: CHAN_18 -> /_CH18
- D20 pad 3: CHAN_19 -> /_CH19
- D21 pad 3: CHAN_20 -> /_CH20
- D22 pad 3: CHAN_21 -> /_CH21
- D23 pad 3: CHAN_22 -> /_CH22
- D24 pad 3: CHAN_23 -> /_CH23
- D25 pad 2: (no net) -> unconnected-(D25-A-Pad2)
- J1 pad 19: CHAN_12 -> /_CH12
- J1 pad 20: CHAN_13 -> /_CH13
- J1 pad 21: CHAN_14 -> /_CH14
- J1 pad 22: CHAN_15 -> /_CH15
- J1 pad 24: CHAN_16 -> /_CH16
- J1 pad 25: CHAN_17 -> /_CH17
- J1 pad 26: CHAN_18 -> /_CH18
- J1 pad 27: CHAN_19 -> /_CH19
- J1 pad 29: CHAN_20 -> /_CH20
- J1 pad 30: (no net) -> unconnected-(J1-RUN-Pad30)
- J1 pad 31: CHAN_21 -> /_CH21
- J1 pad 32: CHAN_22 -> /_CH22
- J1 pad 33: (no net) -> unconnected-(J1-AGND-Pad33)
- J1 pad 34: CHAN_23 -> /_CH23
- J1 pad 35: (no net) -> unconnected-(J1-ADC_VREF-Pad35)_0
- J1 pad 37: (no net) -> unconnected-(J1-3V3_EN-Pad37)_0
- J1 pad 39: (no net) -> unconnected-(J1-VSYS-Pad39)
- J2 pad 10: $1N7399 -> /CH13
- J2 pad 12: $1N7403 -> /CH14
- J2 pad 14: $1N7407 -> /CH15
- J2 pad 16: $1N7411 -> /CH16
- J2 pad 18: $1N7415 -> /CH17
- J2 pad 20: $1N7419 -> /CH18
- J2 pad 22: $1N7423 -> /CH19
- J2 pad 24: $1N7427 -> /CH20
- J2 pad 26: $1N7431 -> /CH21
- J2 pad 28: $1N7435 -> /CH22
- J2 pad 30: $1N7439 -> /CH23
- J2 pad 8: $1N7395 -> /CH12
- R13 pad 1: $1N7395 -> /_CH12
- R13 pad 2: CHAN_12 -> /CH12
- R14 pad 1: $1N7399 -> /_CH13
- R14 pad 2: CHAN_13 -> /CH13
- R15 pad 1: $1N7403 -> /_CH14
- R15 pad 2: CHAN_14 -> /CH14
- R16 pad 1: $1N7407 -> /_CH15
- R16 pad 2: CHAN_15 -> /CH15
- R17 pad 1: $1N7411 -> /_CH16
- R17 pad 2: CHAN_16 -> /CH16
- R18 pad 1: $1N7415 -> /_CH17
- R18 pad 2: CHAN_17 -> /CH17
- R19 pad 1: $1N7419 -> /_CH18
- R19 pad 2: CHAN_18 -> /CH18
- R20 pad 1: $1N7423 -> /_CH19
- R20 pad 2: CHAN_19 -> /CH19
- R21 pad 1: $1N7427 -> /_CH20
- R21 pad 2: CHAN_20 -> /CH20
- R22 pad 1: $1N7431 -> /_CH21
- R22 pad 2: CHAN_21 -> /CH21
- R23 pad 1: $1N7435 -> /_CH22
- R23 pad 2: CHAN_22 -> /CH22
- R24 pad 1: $1N7439 -> /_CH23
- R24 pad 2: CHAN_23 -> /CH23
Routing:
- net CHAN_12: track 43.8 -> 0.00 mm
- net /_CH12: track 0.00 -> 43.8 mm
- net CHAN_15: track 43.3 -> 0.00 mm
- net /_CH15: track 0.00 -> 43.3 mm
- net CHAN_14: track 43.3 -> 0.00 mm
- net /_CH14: track 0.00 -> 43.3 mm
- net CHAN_13: track 43.3 -> 0.00 mm
- net /_CH13: track 0.00 -> 43.3 mm
- net CHAN_19: track 43.2 -> 0.00 mm
- net /_CH19: track 0.00 -> 43.2 mm
- net CHAN_17: track 43.2 -> 0.00 mm
- net /_CH17: track 0.00 -> 43.2 mm
- net CHAN_16: track 43.2 -> 0.00 mm
- net /_CH16: track 0.00 -> 43.2 mm
- net CHAN_18: track 43.2 -> 0.00 mm
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Other:
- board text added: "trace lengths 38.46 + 4.84 = 43.3 41.64 + 1.66 = 43.3"
- board text removed: "trace lengths pi to diode to resistor 38.46 + 4.84 = 43.3 41.64 + 1.66 = 43.3"
