File: PCB/peeko_3v3.kicad_pcb (KiCad board)
At the start: 2 copper layers, 21.1 x 51.3 mm, 6 parts, among them J1 Raspberry PI Pico, J2 Conn_02x15_Odd_Even, J3 Conn_01x02_Pin, J4 Conn_01x02_Pin

Commit message: minor
Parts:
- moved D1 14.2 mm to (148.6, 132.1)
- moved J1 14.2 mm to (152.4, 114.3)
- moved J4 14.2 mm to (148.6, 99.1)
- moved R1 14.2 mm to (146.7, 134.6)
- moved J2 14.2 mm to (151.1, 129.5)
- moved J3 14.2 mm to (146.1, 129.5)
Other:
- board text added: "14.55 19.63"
- board text removed: "14.55mm 19.63mm"
