File: PCB/peeko_3v3.kicad_sch (KiCad schematic)
At the start: 6 parts, among them J1 Rasberry PI Pico, J2 Conn_02x15_Odd_Even, J3 Conn_01x02_Pin, J4 Conn_01x02_Pin

Commit message: minor
Other:
- moved on the sheet: J2
Changed lines of the file:
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@@
 	(wire
 		(pts
-			(xy 95.25 106.68) (xy 95.25 127)
+			(xy 95.25 110.49) (xy 95.25 127)
 		)
 		(stroke
@@
 	)
 	(label "CH6"
-		(at 95.25 91.44 180)
+		(at 95.25 95.25 180)
 		(fields_autoplaced yes)
 		(effects
@@
 	)
 	(label "CH7"
-		(at 95.25 93.98 180)
+		(at 95.25 97.79 180)
 		(fields_autoplaced yes)
 		(effects
@@
 	)
 	(label "CH17"
-		(at 107.95 91.44 0)
+		(at 107.95 95.25 0)
 		(fields_autoplaced yes)
 		(effects
@@
 	)
 	(label "CH20"
-		(at 107.95 83.82 0)
+		(at 107.95 87.63 0)
 		(fields_autoplaced yes)
 		(effects
@@
 	)
 	(label "CH2"
-		(at 95.25 81.28 180)
+		(at 95.25 85.09 180)
 		(fields_autoplaced yes)
 		(effects
@@
 	)
 	(label "CH4"
-		(at 95.25 86.36 180)
+		(at 95.25 90.17 180)
 		(fields_autoplaced yes)
 		(effects
@@
 	)
 	(label "CH3"
-		(at 95.25 83.82 180)
+		(at 95.25 87.63 180)
 		(fields_autoplaced yes)
 		(effects
@@
 	)
 	(label "CH18"
-		(at 107.95 88.9 0)
+		(at 107.95 92.71 0)
 		(fields_autoplaced yes)
 		(effects
@@
 	)
 	(label "CH23"
-		(at 107.95 76.2 0)
+		(at 107.95 80.01 0)
 		(fields_autoplaced yes)
 		(effects
@@
 	)
 	(label "CH14"
-		(at 107.95 99.06 0)
+		(at 107.95 102.87 0)
 		(fields_autoplaced yes)
 		(effects
@@
 	)
 	(label "CH11"
-		(at 95.25 104.14 180)
+		(at 95.25 107.95 180)
 		(fields_autoplaced yes)
 		(effects
@@
 		)
 	)
-	(label "CH{0..23}"
-		(at 127 63.5 0)
-		(fields_autoplaced yes)
-		(effects
-			(font
-				(size 1.27 1.27)
-			)
-			(justify left bottom)
-		)
-	)
 	(label "CHAIN"
 		(at 133.35 142.24 0)
@@
 	)
 	(label "CH16"
-		(at 107.95 93.98 0)
+		(at 107.95 97.79 0)
 		(fields_autoplaced yes)
 		(effects
@@
 	)
 	(label "CH22"
-		(at 107.95 78.74 0)
+		(at 107.95 82.55 0)
 		(fields_autoplaced yes)
 		(effects
@@
 	)
 	(label "TRIGGER"
-		(at 95.25 106.68 180)
+		(at 95.25 110.49 180)
 		(fields_autoplaced yes)
 		(effects
@@
 	)
 	(label "CH12"
-		(at 107.95 104.14 0)
+		(at 107.95 107.95 0)
 		(fields_autoplaced yes)
 		(effects
@@
 	)
 	(label "CH19"
-		(at 107.95 86.36 0)
+		(at 107.95 90.17 0)
 		(fields_autoplaced yes)
 		(effects
@@
 	)
 	(label "CH9"
-		(at 95.25 99.06 180)
+		(at 95.25 102.87 180)
 		(fields_autoplaced yes)
 		(effects
@@
 	)
 	(label "CH8"
-		(at 95.25 96.52 180)
+		(at 95.25 100.33 180)
 		(fields_autoplaced yes)
 		(effects
@@
 	)
 	(label "CH21"
-		(at 107.95 81.28 0)
+		(at 107.95 85.09 0)
 		(fields_autoplaced yes)
 		(effects
@@
 	)
 	(label "CH0"
-		(at 95.25 76.2 180)
+		(at 95.25 80.01 180)
 		(fields_autoplaced yes)
 		(effects
@@
 	)
 	(label "CH5"
-		(at 95.25 88.9 180)
+		(at 95.25 92.71 180)
 		(fields_autoplaced yes)
 		(effects
@@
 	)
 	(label "CH10"
-		(at 95.25 101.6 180)
+		(at 95.25 105.41 180)
 		(fields_autoplaced yes)
 		(effects
@@
 	)
 	(label "CH13"
-		(at 107.95 101.6 0)
+		(at 107.95 105.41 0)
 		(fields_autoplaced yes)
 		(effects
@@
 	)
 	(label "CH1"
-		(at 95.25 78.74 180)
+		(at 95.25 82.55 180)
 		(fields_autoplaced yes)
 		(effects
@@
 	)
 	(label "CH15"
-		(at 107.95 96.52 0)
+		(at 107.95 100.33 0)
 		(fields_autoplaced yes)
 		(effects
@@
 		(dnp no)
 		(property "Reference" "J1"
+			(at 177.8 63.5 0)
+			(effects
+				(font
+					(size 1.27 1.27)
+				)
+			)
+		)
+		(property "Value" "Rasberry PI Pico"
 			(at 177.8 65.532 0)
-			(effects
-				(font
-					(size 1.27 1.27)
-				)
-			)
-		)
-		(property "Value" "Rasberry PI Pico"
-			(at 177.8 67.564 0)
 			(effects
 				(font
@@
 	(symbol
 		(lib_id "power:GND")
-		(at 107.95 106.68 0)
+		(at 107.95 110.49 0)
 		(unit 1)
 		(exclude_from_sim no)
@@
 		(fields_autoplaced yes)
 		(property "Reference" "#PWR04"
-			(at 107.95 113.03 0)
+			(at 107.95 116.84 0)
 			(effects
 				(font
@@
 		)
 		(property "Value" "GND"
-			(at 107.95 111.76 0)
+			(at 107.95 115.57 0)
 			(effects
 				(font
@@
 		)
 		(property "Footprint" ""
-			(at 107.95 106.68 0)
+			(at 107.95 110.49 0)
 			(effects
 				(font
@@
 		)
 		(property "Datasheet" ""
-			(at 107.95 106.68 0)
+			(at 107.95 110.49 0)
 			(effects
 				(font
@@
 		)
 		(property "Description" "Power symbol creates a global label with name \"GND\" , ground"
-			(at 107.95 106.68 0)
+			(at 107.95 110.49 0)
 			(effects
 				(font
@@
 	(symbol
 		(lib_id "Connector_Generic:Conn_02x13_Odd_Even")
-		(at 100.33 91.44 0)
+		(at 100.33 95.25 0)
 		(mirror x)
 		(unit 1)
@@
 		(dnp no)
 		(property "Reference" "J2"
-			(at 101.6 66.802 0)
+			(at 101.6 70.612 0)
 			(effects
 				(font
@@
 		)
 		(property "Value" "Conn_02x15_Odd_Even"
-			(at 101.854 69.342 0)
+			(at 101.854 73.152 0)
 			(effects
 				(font
@@
 		)
 		(property "Footprint" "Connector_IDC:IDC-Header_2x13_P2.54mm_Horizontal"
-			(at 100.33 91.44 0)
+			(at 100.33 95.25 0)
 			(effects
 				(font
@@
 		)
 		(property "Datasheet" "~"
-			(at 100.33 91.44 0)
+			(at 100.33 95.25 0)
 			(effects
 				(font
@@
 		)
 		(property "Description" "Generic connector, double row, 02x13, odd/even pin numbering scheme (row 1 odd numbers, row 2 even numbers), script generated (kicad-library-utils/schlib/autogen/connector/)"
-			(at 100.33 91.44 0)
-			(effects
-				(font
+			(at 100.33 95.25 0)
+			(effects
+				(font
