File: PCB/peeko_jy.kicad_sch (KiCad schematic)
At the start: 54 parts, among them J1 Rasberry PI Pico, J2 Conn_02x15_Odd_Even, J3 Conn_01x02_Pin, J4 Conn_01x02_Pin

Commit message: minor
Other:
- title: peeko -> peeko_jy
Changed lines of the file:
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@@
 	(paper "A4")
 	(title_block
-		(title "peeko")
-		(date "2024-09-16")
+		(title "peeko_jy")
+		(date "2024-09-21")
 		(rev "001")
 		(comment 1 "github.com/bkw777/peeko")
