File: PCB/peeko.kicad_sch (KiCad schematic)
At the start: 6 parts, among them J1 Rasberry PI Pico, J2 Conn_02x15_Odd_Even, J3 Conn_01x02_Pin, J4 Conn_01x02_Pin

Commit message: schematic for JY board, remove all but PCBs
Changed lines of the file:
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@@
-	(wire
-		(pts
-			(xy 107.95 88.9) (xy 113.03 88.9)
-		)
-		(stroke
-			(width 0)
-			(type default)
-		)
-	)
 	(wire
 		(pts
@@
 	(wire
 		(pts
-			(xy 107.95 81.28) (xy 113.03 81.28)
-		)
-		(stroke
-			(width 0)
-			(type default)
-		)
-	)
-	(wire
-		(pts
 			(xy 152.4 101.6) (xy 160.02 101.6)
 		)
@@
 	(wire
 		(pts
-			(xy 107.95 86.36) (xy 113.03 86.36)
-		)
-		(stroke
-			(width 0)
-			(type default)
-		)
-	)
-	(wire
-		(pts
 			(xy 195.58 76.2) (xy 203.2 76.2)
 		)
@@
 	(wire
 		(pts
-			(xy 107.95 76.2) (xy 113.03 76.2)
-		)
-		(stroke
-			(width 0)
-			(type default)
-		)
-	)
-	(wire
-		(pts
 			(xy 133.35 127) (xy 133.35 142.24)
 		)
@@
 	(wire
 		(pts
-			(xy 107.95 99.06) (xy 113.03 99.06)
-		)
-		(stroke
-			(width 0)
-			(type default)
-		)
-	)
-	(wire
-		(pts
 			(xy 203.2 101.6) (xy 203.2 114.3)
 		)
@@
 	(wire
 		(pts
-			(xy 107.95 93.98) (xy 113.03 93.98)
-		)
-		(stroke
-			(width 0)
-			(type default)
-		)
-	)
-	(wire
-		(pts
-			(xy 107.95 101.6) (xy 113.03 101.6)
-		)
-		(stroke
-			(width 0)
-			(type default)
-		)
-	)
-	(wire
-		(pts
 			(xy 133.35 144.78) (xy 139.7 144.78)
 		)
@@
 	(wire
 		(pts
-			(xy 107.95 96.52) (xy 113.03 96.52)
-		)
-		(stroke
-			(width 0)
-			(type default)
-		)
-	)
-	(wire
-		(pts
 			(xy 118.11 127) (xy 133.35 127)
 		)
@@
 	(wire
 		(pts
-			(xy 107.95 91.44) (xy 113.03 91.44)
-		)
-		(stroke
-			(width 0)
-			(type default)
-		)
-	)
-	(wire
-		(pts
 			(xy 127 144.78) (xy 133.35 144.78)
 		)
@@
 	(wire
 		(pts
-			(xy 107.95 78.74) (xy 113.03 78.74)
-		)
-		(stroke
-			(width 0)
-			(type default)
-		)
-	)
-	(wire
-		(pts
 			(xy 133.35 71.12) (xy 160.02 71.12)
 		)
@@
 		)
 		(stroke
-			(width 0)
-			(type default)
-		)
-	)
-	(wire
-		(pts
-			(xy 107.95 83.82) (xy 113.03 83.82)
-		)
-		(stroke
-			(width 0)
-			(type default)
-		)
-	)
-	(wire
-		(pts
-			(xy 107.95 104.14) (xy 113.03 104.14)
-		)
-		(stroke

Commit message: fixup local symbols, footprints, models, move power traces inboard
Parts:
- J2: footprint Connector_IDC:IDC-Header_2x15_P2.54mm_Horizontal -> 000_LOCAL:IDC-Header_2x15_P2.54mm_Horizontal
Changed lines of the file:
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@@
 			)
 		)
-		(property "Footprint" "Connector_IDC:IDC-Header_2x15_P2.54mm_Horizontal"
+		(property "Footprint" "000_LOCAL:IDC-Header_2x15_P2.54mm_Horizontal"
 			(at 100.33 93.98 0)
 			(effects
