File: PCB/peeko+.kicad_sch (KiCad schematic)
At the start: 25 parts, among them J1 Rasberry PI Pico, J2 Conn_02x15_Odd_Even, J3 Conn_01x02_Pin, J4 Conn_01x02_Pin, U1 TXU0104, U2 TXU0104, U3 TXU0104, U4 TXU0104, U5 TXU0104, U6 TXU0104

Commit message: peeko+ housing render
Parts:
- added N1: Housing, 000_LOCAL:peeko+_housing, symbol 000_LOCAL:Housing
Changed lines of the file:
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@@
+	)
+	(symbol
+		(lib_id "000_LOCAL:Housing")
+		(at 50.8 177.8 0)
+		(unit 1)
+		(exclude_from_sim yes)
+		(in_bom yes)
+		(on_board yes)
+		(dnp no)
+		(fields_autoplaced yes)
+		(property "Reference" "N1"
+			(at 54.61 176.8474 0)
+			(effects
+				(font
+					(size 1.27 1.27)
+				)
+				(justify left)
+			)
+		)
+		(property "Value" "Housing"
+			(at 54.61 179.3874 0)
+			(effects
+				(font
+					(size 1.27 1.27)
+				)
+				(justify left)
+			)
+		)
+		(property "Footprint" "000_LOCAL:peeko+_housing"
+			(at 52.07 176.53 0)
+			(effects
+				(font
+					(size 1.27 1.27)
+				)
+				(hide yes)
+			)
+		)
+		(property "Datasheet" "~"
+			(at 52.07 176.53 0)
+			(effects
+				(font
+					(size 1.27 1.27)
+				)
+				(hide yes)
+			)
+		)
+		(property "Description" "Housing"
+			(at 50.8 177.8 0)
+			(effects
+				(font
+					(size 1.27 1.27)
+				)
+				(hide yes)
+			)
+		)
+		(instances
+			(project ""
+				(path "/9dbd0e01-4650-4cf8-82d3-a69ef2ebdc12"
+					(reference "N1")
+					(unit 1)
+				)
+			)
+		)
 	)
 	(symbol
