File: PCB/PEEKO-Brute.kicad_pcb (KiCad board)
At the start: 2 copper layers, 52.1 x 43.2 mm, 61 parts, among them J1 Rasberry PI Pico, J2 Conn_02x15_Odd_Even, J3 Conn_01x02_Pin, J4 Conn_01x02_Pin

Commit message: forgotten fillet track on brute
Routing:
- net GND: vias 119 -> 121
